Commit message: fix : made the arms straight

File: description/botzilla_qbot.urdf (robot description, URDF)
Before this commit: robot botzilla_qbot, 9 links, 8 joints
Joints:
- joint arm_left_joint: origin xyz=0.18 0.06 -0.01 rpy=0 0 0.3 -> xyz=0.18 0.08 -0.01 rpy=0 0 0
- joint arm_right_joint: origin xyz=0.18 -0.06 -0.01 rpy=0 0 -0.3 -> xyz=0.18 -0.08 -0.01 rpy=0 0 0
- joint base_joint: origin xyz=0 0 0.05 rpy=0 0 0 -> xyz=0 0 0.00 rpy=0 0 0
